File: PCB/GBAKicad.kicad_pcb (KiCad board)
At the start: 2 copper layers, 132.9 x 88.4 mm, 67 parts, among them J1 USB_C_Receptacle_USB2.0_16P, J2 BATT_Conn, J3 Jumper, J4 OLED_Conn, Q2 PMOS, SW1 EN, SW10 BTN_R, SW11 BTN_X, SW12 BTN_A, SW13 BTN_B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

Commit message: CAD files
Parts:
- moved H2 27.0 mm to (194.2, 105.8)
- moved H4 24.5 mm to (106.9, 107.1)
- moved H1 5.87 mm to (205.6, 98.0)
- moved H3 2.77 mm to (92.8, 97.7)
Other:
- board size 132.9 x 88.4 mm -> 132.9 x 71.3 mm
Changed lines of the file:
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@@
 	(footprint "MountingHole:MountingHole_3.2mm_M3"
 		(layer "F.Cu")
-		(at 201.51 131.8)
+		(at 194.2 105.8)
 		(descr "Mounting Hole 3.2mm, M3, no annular, generated by kicad-footprint-generator mountinghole.py")
 		(tags "mountinghole M3")
@@
 	(footprint "MountingHole:MountingHole_3.2mm_M3"
 		(layer "F.Cu")
-		(at 211.47 97.97)
+		(at 205.6 97.97)
 		(descr "Mounting Hole 3.2mm, M3, no annular, generated by kicad-footprint-generator mountinghole.py")
 		(tags "mountinghole M3")
@@
 	(footprint "MountingHole:MountingHole_3.2mm_M3"
 		(layer "F.Cu")
-		(at 99.73 130.57)
+		(at 106.9 107.1)
 		(descr "Mounting Hole 3.2mm, M3, no annular, generated by kicad-footprint-generator mountinghole.py")
 		(tags "mountinghole M3")
@@
 	(footprint "MountingHole:MountingHole_3.2mm_M3"
 		(layer "F.Cu")
-		(at 90.91 99.73)
+		(at 92.8 97.7)
 		(descr "Mounting Hole 3.2mm, M3, no annular, generated by kicad-footprint-generator mountinghole.py")
 		(tags "mountinghole M3")
@@
 		(layer "Edge.Cuts")
 	)
-	(gr_curve
-		(pts
-			(xy 84.64 104.495) (xy 84.64 149.745) (xy 108.82 146.56) (xy 118.84 122.655)
-		)
+	(gr_line
+		(start 118.84 122.655)
+		(end 84.64 104.495)
 		(stroke
 			(width 0.05)
@@
 	)
 	(gr_line
-		(start 214.77 72.92)
+		(start 183.37 122.41)
 		(end 217.57 104.25)
 		(stroke
@@
 		(layer "Edge.Cuts")
 	)
-	(gr_curve
-		(pts
-			(xy 217.57 104.25) (xy 217.57 149.5) (xy 193.39 146.315) (xy 183.37 122.41)
-		)
+	(gr_line
+		(start 214.77 72.92)
+		(end 217.57 104.25)
 		(stroke
 			(width 0.05)
